File: Kicad/PC-8001_RAM.sch (KiCad schematic (older format))
At the start: 12 parts, among them J1 PC-8001 BUS, J2 PC-8001 BUS, U1 GAL22V10, U2 62256, U3 CY7C199

Commit message: Add files via upload
Parts:
- added C4: 0.1uF, Capacitor_THT:C_Rect_L4.0mm_W2.5mm_P2.50mm, symbol Device:C
- added U4: 74LS04, Package_DIP:DIP-14_W7.62mm_LongPads, symbol 74xx:74LS04
Connections:
- wire segments 221 -> 235
- no-connect marks 0 -> 5
Other:
- moved on the sheet: C2, U2, U3

Commit message: Add files via upload
Connections:
- net labels added: ~WE-RAM
Changed lines of the file:
@@
 Title "PC-8001_RAM"
 Date "2025-08-16"
-Rev "Rev1.3"
+Rev "Rev1.4"
 Comp ""
 Comment1 ""
@@
 LATCHRD
 Text Label 5200 1950 0    50   ~ 0
-~WE
+~WE-RAM
 Text Label 5200 2050 0    50   ~ 0
 ~CS
@@
 ~CS
 Text Label 9600 2500 0    50   ~ 0
-~WE
+~WE-RAM
 $Comp
 L Device:C C1
@@
 ~CS
 Text Label 9150 5700 0    50   ~ 0
-~WE
+~WE-RAM
 $Comp
 L power:+5V #PWR07
